File: KiCadTraining.kicad_pcb (KiCad board)
At the start: 2 copper layers, 83 parts, among them Q1 2SC1815, Q10 2SC1815, Q11 2SA1015, Q12 2SA1015, Q13 2SC1815, Q14 2SC1815, Q15 2SC1815, Q16 2SC1815, Q17 2SC1815, Q18 2SC1815, Q19 2SC1815, Q2 2SC1815, Q20 2SC1815, Q21 2SC1815, Q22 2SC1815, Q23 2SC1815, Q24 2SC1815, Q25 2SC1815, Q3 2SC1815, Q4 2SC1815, Q5 2SA1015, Q6 2SA1015, Q7 2SA1015, Q8 2SA1015, Q9 2SC1815, SW1 SW_Push_Dual, SW2 SW_Push_Dual, SW3 SW_Push_Dual, SW4 SW_Push_Dual, SW5 SW_Push_Dual, U1 STM32NUCLEO-L476RG, U2 A-2301SR, U3 A-2301SR, U4 A-2301SR, U5 A-2301SR, U6 A-2301SR, U7 A-2301SR

Commit message: 部品レイアウトを合理化
Parts:
- moved SW4 65.2 mm to (48.3, 47.0)
- moved SW1 65.0 mm to (48.3, 33.0)
- moved Q13 59.3 mm to (207.0, 110.5)
- moved Q14 59.3 mm to (207.0, 119.4)
- moved Q15 59.3 mm to (207.0, 128.3)
- moved Q16 59.3 mm to (207.0, 137.2)
- moved Q17 59.3 mm to (207.0, 146.1)
- moved Q18 59.3 mm to (207.0, 154.9)
- moved Q19 59.3 mm to (207.0, 163.8)
- moved R19 59.3 mm to (199.4, 110.5)
- moved R20 59.3 mm to (199.4, 119.4)
- moved R21 59.3 mm to (199.4, 128.3)
- moved R22 59.3 mm to (199.4, 137.2)
- moved R23 59.3 mm to (199.4, 146.1)
- moved R24 59.3 mm to (199.4, 154.9)
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